Commit message: gengxin

File: install/mower_description/share/mower_description/urdf/mower.urdf (robot description, URDF)
Before this commit: robot mower, 12 links, 11 joints
Links:
- added link blade1_link, mass 0.1; collision box size=0.18 0.01 0.005; visual box size=0.18 0.01 0.005
- added link blade2_link, mass 0.1; collision box size=0.18 0.01 0.005; visual box size=0.18 0.01 0.005
- added link blade3_link, mass 0.1; collision box size=0.18 0.01 0.005; visual box size=0.18 0.01 0.005
- added link cutting_motor_link, mass 0.5; collision cylinder length=0.03 radius=0.03; visual cylinder length=0.03 radius=0.03
- link base_link: geometry collision box size=0.5665 0.37 0.15; visual box size=0.48 0.015 0.025
- link bumper_link: geometry collision box size=0.1 0.3 0.05; visual box size=0.1 0.3 0.05
- link front_left_caster: geometry collision cylinder length=0.03 radius=0.045; visual cylinder length=0.03 radius=0.045
- link front_right_caster: geometry collision cylinder length=0.03 radius=0.045; visual cylinder length=0.03 radius=0.045
- link laser_link: geometry visual box size=0.1 0.1 0.05; visual box size=0.102 0.102 0.012
- link left_wheel: geometry collision cylinder length=0.05 radius=0.11; visual cylinder length=0.05 radius=0.11
- link right_wheel: geometry collision cylinder length=0.05 radius=0.11; visual cylinder length=0.05 radius=0.11
- link ultrasonic_link: geometry visual box size=0.005 0.02 0.02; visual box size=0.04 0.02 0.02
Joints:
- added joint blade1_joint: type fixed, parent cutting_motor_link, child blade1_link, origin xyz=0 0 -0.016 rpy=0 0 0
- added joint blade2_joint: type fixed, parent cutting_motor_link, child blade2_link, origin xyz=0 0 -0.016 rpy=0 0 0
- added joint blade3_joint: type fixed, parent cutting_motor_link, child blade3_link, origin xyz=0 0 -0.016 rpy=0 0 0
- added joint blade_joint: type continuous, parent base_link, child cutting_motor_link, origin xyz=0.12 0 -0.01 rpy=0 0 0, axis 0 0 1, limit effort=50 velocity=80
- joint bumper_joint: origin xyz=0 0 0 rpy=0 0 0 -> xyz=0.12 0 0 rpy=0 0 0
- joint camera_joint: origin xyz=0.22 0 0.165 rpy=0 0 0 -> xyz=0.34 0 0.165 rpy=0 0 0
- joint front_left_caster_joint: origin xyz=0.15 0.18 0.05 rpy=0 0 0 -> xyz=0.30 0.0925 -0.035 rpy=0 0 0
- joint front_right_caster_joint: origin xyz=0.15 -0.18 0.05 rpy=0 0 0 -> xyz=0.30 -0.0925 -0.035 rpy=0 0 0
- joint imu_joint: origin xyz=0 0 0.075 rpy=0 0 0 -> xyz=0.12 0 0.075 rpy=0 0 0
- joint left_wheel_joint: origin xyz=-0.2 0.2 0.07 rpy=0 0 0 -> xyz=0 0.16 0.03 rpy=0 0 0
- joint lidar_mast_joint: origin xyz=0.0 0.0 0.17 rpy=0 0 0 -> xyz=0.12 0.0 0.17 rpy=0 0 0
- joint right_wheel_joint: origin xyz=-0.2 -0.2 0.07 rpy=0 0 0 -> xyz=0 -0.16 0.03 rpy=0 0 0
- joint ultrasonic_joint: origin xyz=0.27 0 0.08 rpy=0 0 0 -> xyz=0.39 0 0.08 rpy=0 0 0
